File: hardware/PCB_Manufacturing/SmartHomeController.kicad_pcb (KiCad board)
At the start: 2 copper layers, 100 x 80 mm, 11 parts, among them Q1 BT136-600E, Q2 BT136-600E, Q3 BT136-600E, Q4 BT136-600E, U1 ESP32-WROOM-32, U2 MOC3021, U3 MOC3021, U4 MOC3021, U5 MOC3021, U6 4N25, U7 AMS1117-5.0

Commit message: Fix code review issues: MOC3021 pin overlap and TRIAC gate net assignments
Co-authored-by: Gokul3611 <177666785+Gokul3611@users.noreply.github.com>
Connections:
- Q3 pad 3: Net-(Q1-Pad3) -> Net-(Q3-Pad3)
- Q4 pad 3: Net-(Q2-Pad3) -> Net-(Q4-Pad3)
- U4 pad 4: Net-(Q1-Pad3) -> Net-(Q3-Pad3)
- U5 pad 4: Net-(Q2-Pad3) -> Net-(Q4-Pad3)
Changed lines of the file:
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@@
     (zones 2)
     (modules 45)
-    (nets 35)
+    (nets 37)
   )
   (page "A3")
@@
   (net 33 "Net-(Q1-Pad3)")
   (net 34 "Net-(Q2-Pad3)")
+  (net 35 "Net-(Q3-Pad3)")
+  (net 36 "Net-(Q4-Pad3)")
   (net_class "Default" "Default net class."
     (clearance 0.2)
@@
       (net 13 "AC_LIVE"))
     (pad "3" thru_hole circle (at 5.08 0) (size 1.8 1.8) (drill 1.0) (layers *.Cu *.Mask)
-      (net 33 "Net-(Q1-Pad3)"))
+      (net 35 "Net-(Q3-Pad3)"))
     (pad "" thru_hole circle (at 0 2) (size 0.5 0.5) (drill 0.5) (layers *.Cu)
       (net 1 "GND") (zone_connect 2))
@@
       (net 13 "AC_LIVE"))
     (pad "3" thru_hole circle (at 5.08 0) (size 1.8 1.8) (drill 1.0) (layers *.Cu *.Mask)
-      (net 34 "Net-(Q2-Pad3)"))
+      (net 36 "Net-(Q4-Pad3)"))
     (pad "" thru_hole circle (at 0 2) (size 0.5 0.5) (drill 0.5) (layers *.Cu)
       (net 1 "GND") (zone_connect 2))
@@
       (net 1 "GND"))
     (pad "4" thru_hole circle (at 7.62 2.54 90) (size 1.6 1.6) (drill 0.8) (layers *.Cu *.Mask)
-      (net 33 "Net-(Q1-Pad3)"))
+      (net 35 "Net-(Q3-Pad3)"))
     (pad "6" thru_hole circle (at 7.62 0 90) (size 1.6 1.6) (drill 0.8) (layers *.Cu *.Mask)
       (net 17 "AC_L3"))
@@
       (net 1 "GND"))
     (pad "4" thru_hole circle (at 7.62 2.54 90) (size 1.6 1.6) (drill 0.8) (layers *.Cu *.Mask)
-      (net 34 "Net-(Q2-Pad3)"))
+      (net 36 "Net-(Q4-Pad3)"))
     (pad "6" thru_hole circle (at 7.62 0 90) (size 1.6 1.6) (drill 0.8) (layers *.Cu *.Mask)
       (net 18 "AC_L4"))
